File: STM32.kicad_sch (KiCad schematic)
At the start: 0 parts

Commit message: till usb debugger - differential pair
Parts:
- added C1, C2, C3, C4, C8: 100n, Package_QFP:LQFP-48_7x7mm_P0.5mm, symbol Device:C
- added C5: 10n, Package_QFP:LQFP-48_7x7mm_P0.5mm, symbol Device:C
- added C6, C7: 1u, Package_QFP:LQFP-48_7x7mm_P0.5mm, symbol Device:C
- added FB1: 120R, Package_LCC:PLCC-84_29.3x29.3mm_P1.27mm, symbol Device:FerriteBead
- added R1: 10K, symbol Device:R
- added SW1: SW_SPDT, Package_SO:SOIC-28W_7.5x17.9mm_P1.27mm, symbol Switch:SW_SPDT
- added U1: STM32F103C8T6, Package_QFP:LQFP-48_7x7mm_P0.5mm, symbol MCU_ST_STM32F1:STM32F103C8Tx
Connections:
- new net: R1.1, SW1.2 (B)
- new net +3.3V: C1.1, C2.1, C3.1, C4.1, C7.1, FB1.2, SW1.3 (C), U1.1 (VBAT), U1.24 (VDD), U1.36 (VDD), U1.48 (VDD)
- new net +3.3VA: C5.1, C6.1, FB1.1, U1.9 (VDDA)
- new net BOOT0: R1.2, U1.44 (BOOT0)
- new net GND: C1.2, C2.2, C3.2, C4.2, C5.2, C6.2, C7.2, C8.2, SW1.1 (A), U1.23 (VSS), U1.35 (VSS), U1.47 (VSS), U1.8 (VSSA)
- new net HSE_IN: U1.5 (PD0)
- new net HSE_OUT: U1.6 (PD1)
- new net NRST: C8.1, U1.7 (NRST)
- new net SWCLK: U1.37 (PA14)
- new net SWDIO: U1.34 (PA13)
- new net USB_D+: U1.33 (PA12)
- new net USB_D-: U1.32 (PA11)
Other:
- company: (none) -> SAYOOJ TECHNOLOGY
- title: (none) -> STM32

Commit message: erc
Parts:
- added C10, C9: 10p, Package_QFP:LQFP-48_7x7mm_P0.5mm, symbol Device:C
- added C11, C12: 22u, Package_QFP:LQFP-48_7x7mm_P0.5mm, symbol Device:C
- added D1: RED, symbol Device:LED
- added J1: USB_B_Micro, Package_DFN_QFN:WDFN-10-1EP_3x3mm_P0.5mm_EP1.8x2.5mm, symbol Connector:USB_B_Micro
- added J2, J3, J4: Conn_01x04_Pin, symbol Connector:Conn_01x04_Pin
- added R2: 1k5, symbol Device:R
- added R3, R4, R5: 1K5, symbol Device:R
- added U2: AMS1117-3.3, Package_TO_SOT_SMD:SOT-223-3_TabPin2, symbol Regulator_Linear:AMS1117-3.3
- added Y1: 16MHz, Package_QFP:LQFP-48_7x7mm_P0.5mm, symbol Device:Crystal_GND24
Connections:
- net +3.3V: now also C12.1, D1.2 (A), U2.2 (VO)
- net +3.3VA: now also J2.1 (Pin_1), J3.1 (Pin_1), J4.1 (Pin_1), R2.1, R4.1, R5.1
- net GND: now also C10.2, C11.2, C12.2, C9.2, J1.5 (GND), J2.4 (Pin_4), J3.4 (Pin_4), J4.4 (Pin_4), R3.2, U2.1 (GND), Y1.2 (G), Y1.4 (G)
- net HSE_IN: now also C9.1, Y1.1
- net HSE_OUT: now also C10.1, Y1.3
- net SWCLK: now also J2.3 (Pin_3)
- net SWDIO: now also J2.2 (Pin_2)
- net SW_BOOT0: now also R1.1, SW1.2 (B)
- net USB_D+: now also J1.3 (D+), R2.2
- net USB_D-: now also J1.2 (D-)
- net I2C2_SCL: now reaches U1.21 (PB10)
- net I2C2_SCL: now also J4.2 (Pin_2), R4.2
- net I2C2_SDA: now reaches U1.22 (PB11)
- net I2C2_SDA: now also J4.3 (Pin_3), R5.2
- net USART1_TX: now reaches U1.42 (PB6)
- net USART1_TX: now also J3.2 (Pin_2)
- net USART1_RX: now reaches U1.43 (PB7)
- net USART1_RX: now also J3.3 (Pin_3)
- new net PWR_LED_K: D1.1 (K), R3.1
- new net VBUS: C11.1, J1.1 (VBUS), U2.3 (VI)
- no-connect marks 0 -> 29
Other:
- note added: "MICROCONTROLLER (AND USB)"
- note added: "POWER SUPPLY"
- note added: "STM32 PCB"
- moved on the sheet: C1, C2, C3, C4, C5, C6, C7, C8, FB1, R1, SW1, U1

Commit message: footprints added
Parts:
- C1, C2, C3, C4, C8: footprint Package_QFP:LQFP-48_7x7mm_P0.5mm -> Capacitor_SMD:C_0402_1005Metric
- C10: footprint Package_QFP:LQFP-48_7x7mm_P0.5mm -> Capacitor_SMD:C_0603_1608Metric_Pad1.08x0.95mm_HandSolder
- C11, C12, C6, C7, C9: footprint Package_QFP:LQFP-48_7x7mm_P0.5mm -> Capacitor_SMD:C_0805_2012Metric
- D1: footprint (none) -> LED_SMD:LED_0603_1608Metric
- FB1: footprint Package_LCC:PLCC-84_29.3x29.3mm_P1.27mm -> Inductor_SMD:L_0603_1608Metric
- J1: footprint Package_DFN_QFN:WDFN-10-1EP_3x3mm_P0.5mm_EP1.8x2.5mm -> Connector_USB:USB_Micro-B_Technik_TWP-4002D-H3
- J2, J3, J4: footprint (none) -> Connector_PinHeader_1.00mm:PinHeader_1x04_P1.00mm_Vertical_SMD_Pin1Right
- R1, R2, R3, R4, R5: footprint (none) -> Resistor_SMD:R_0402_1005Metric
- SW1: footprint Package_SO:SOIC-28W_7.5x17.9mm_P1.27mm -> Button_Switch_SMD:SW_SPST_CK_KMS2xxG
- Y1: footprint Package_QFP:LQFP-48_7x7mm_P0.5mm -> Crystal:Crystal_SMD_2016-4Pin_2.0x1.6mm
Changed lines of the file:
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@@
 			)
 		)
-		(property "Footprint" ""
+		(property "Footprint" "LED_SMD:LED_0603_1608Metric"
 			(at 63.5 40.64 0)
 			(hide yes)
@@
 			)
 		)
-		(property "Footprint" "Package_QFP:LQFP-48_7x7mm_P0.5mm"
+		(property "Footprint" "Capacitor_SMD:C_0805_2012Metric"
 			(at 227.0252 53.34 0)
 			(hide yes)
@@
 			)
 		)
-		(property "Footprint" "Package_QFP:LQFP-48_7x7mm_P0.5mm"
+		(property "Footprint" "Capacitor_SMD:C_0805_2012Metric"
 			(at 140.6652 104.14 0)
 			(hide yes)
@@
 			)
 		)
-		(property "Footprint" "Package_QFP:LQFP-48_7x7mm_P0.5mm"
+		(property "Footprint" "Capacitor_SMD:C_0402_1005Metric"
 			(at 181.3052 53.34 0)
 			(hide yes)
@@
 			)
 		)
-		(property "Footprint" "Package_LCC:PLCC-84_29.3x29.3mm_P1.27mm"
+		(property "Footprint" "Inductor_SMD:L_0603_1608Metric"
 			(at 238.76 47.498 90)
 			(hide yes)
@@
 			)
 		)
-		(property "Footprint" ""
+		(property "Footprint" "Connector_PinHeader_1.00mm:PinHeader_1x04_P1.00mm_Vertical_SMD_Pin1Right"
 			(at 241.3 109.22 0)
 			(hide yes)
@@
 			)
 		)
-		(property "Footprint" "Package_QFP:LQFP-48_7x7mm_P0.5mm"
+		(property "Footprint" "Capacitor_SMD:C_0805_2012Metric"
 			(at 28.9052 52.07 0)
 			(hide yes)
@@
 			)
 		)
-		(property "Footprint" ""
+		(property "Footprint" "Resistor_SMD:R_0402_1005Metric"
 			(at 158.242 130.81 90)
 			(hide yes)
@@
 			)
 		)
-		(property "Footprint" "Package_QFP:LQFP-48_7x7mm_P0.5mm"
+		(property "Footprint" "Capacitor_SMD:C_0402_1005Metric"
 			(at 158.4452 53.34 0)
 			(hide yes)
@@
 			)
 		)
-		(property "Footprint" "Package_SO:SOIC-28W_7.5x17.9mm_P1.27mm"
+		(property "Footprint" "Button_Switch_SMD:SW_SPST_CK_KMS2xxG"
 			(at 152.4 68.58 0)
 			(hide yes)
@@
 			)
 		)
-		(property "Footprint" "Package_QFP:LQFP-48_7x7mm_P0.5mm"
+		(property "Footprint" "Capacitor_SMD:C_0805_2012Metric"
 			(at 247.3452 53.34 0)
 			(hide yes)
@@
 			)
 		)
-		(property "Footprint" "Package_QFP:LQFP-48_7x7mm_P0.5mm"
+		(property "Footprint" "Capacitor_SMD:C_0402_1005Metric"
 			(at 126.6952 71.12 0)
 			(hide yes)
@@
 			)
 		)
-		(property "Footprint" ""
+		(property "Footprint" "Resistor_SMD:R_0402_1005Metric"
 			(at 167.64 70.358 90)
 			(hide yes)
@@
 			)
 		)
-		(property "Footprint" ""
+		(property "Footprint" "Resistor_SMD:R_0402_1005Metric"
 			(at 149.352 130.81 90)
 			(hide yes)
@@
 			)
 		)
-		(property "Footprint" ""
+		(property "Footprint" "Resistor_SMD:R_0402_1005Metric"
 			(at 233.172 86.36 90)
 			(hide yes)
@@
 			)
 		)
-		(property "Footprint" "Package_QFP:LQFP-48_7x7mm_P0.5mm"
+		(property "Footprint" "Crystal:Crystal_SMD_2016-4Pin_2.0x1.6mm"
 			(at 151.13 91.44 0)
 			(hide yes)
@@
 			)
 		)
-		(property "Footprint" "Package_QFP:LQFP-48_7x7mm_P0.5mm"
+		(property "Footprint" "Capacitor_SMD:C_0603_1608Metric_Pad1.08x0.95mm_HandSolder"
 			(at 163.5252 104.14 0)
 			(hide yes)
@@
 			)
 		)
-		(property "Footprint" ""
+		(property "Footprint" "Connector_PinHeader_1.00mm:PinHeader_1x04_P1.00mm_Vertical_SMD_Pin1Right"
 			(at 134.62 119.38 0)
 			(hide yes)
@@
 			)
 		)
-		(property "Footprint" "Package_QFP:LQFP-48_7x7mm_P0.5mm"
+		(property "Footprint" "Capacitor_SMD:C_0402_1005Metric"
 			(at 147.0152 53.34 0)
 			(hide yes)
@@
 			)
 		)
-		(property "Footprint" "Package_DFN_QFN:WDFN-10-1EP_3x3mm_P0.5mm_EP1.8x2.5mm"
+		(property "Footprint" "Connector_USB:USB_Micro-B_Technik_TWP-4002D-H3"
 			(at 257.81 91.44 0)
 			(hide yes)
@@
 			)
 		)
-		(property "Footprint" "Package_QFP:LQFP-48_7x7mm_P0.5mm"
+		(property "Footprint" "Capacitor_SMD:C_0402_1005Metric"
 			(at 169.8752 53.34 0)
 			(hide yes)
@@
 			)
 		)
-		(property "Footprint" ""
+		(property "Footprint" "Resistor_SMD:R_0402_1005Metric"
 			(at 69.342 45.72 90)
 			(hide yes)
@@
 			)
 		)
-		(property "Footprint" ""
+		(property "Footprint" "Connector_PinHeader_1.00mm:PinHeader_1x04_P1.00mm_Vertical_SMD_Pin1Right"
 			(at 134.62 135.89 0)
 			(hide yes)
@@
 			)
 		)
-		(property "Footprint" "Package_QFP:LQFP-48_7x7mm_P0.5mm"
+		(property "Footprint" "Capacitor_SMD:C_0805_2012Metric"
 			(at 56.8452 52.07 0)
 			(hide yes)

Commit message: wrong foot prints
Parts:
- C10: footprint Capacitor_SMD:C_0603_1608Metric_Pad1.08x0.95mm_HandSolder -> Capacitor_SMD:C_0402_1005Metric
- C5: footprint Package_QFP:LQFP-48_7x7mm_P0.5mm -> Capacitor_SMD:C_0402_1005Metric
- C6, C7: footprint Capacitor_SMD:C_0805_2012Metric -> Capacitor_SMD:C_0402_1005Metric
Changed lines of the file:
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@@
 			)
 		)
-		(property "Footprint" "Capacitor_SMD:C_0805_2012Metric"
+		(property "Footprint" "Capacitor_SMD:C_0402_1005Metric"
 			(at 227.0252 53.34 0)
 			(hide yes)
@@
 			)
 		)
-		(property "Footprint" "Capacitor_SMD:C_0805_2012Metric"
+		(property "Footprint" "Capacitor_SMD:C_0402_1005Metric"
 			(at 247.3452 53.34 0)
 			(hide yes)
@@
 			)
 		)
-		(property "Footprint" "Capacitor_SMD:C_0603_1608Metric_Pad1.08x0.95mm_HandSolder"
+		(property "Footprint" "Capacitor_SMD:C_0402_1005Metric"
 			(at 163.5252 104.14 0)
 			(hide yes)
@@
 			)
 		)
-		(property "Footprint" "Package_QFP:LQFP-48_7x7mm_P0.5mm"
+		(property "Footprint" "Capacitor_SMD:C_0402_1005Metric"
 			(at 215.5952 53.34 0)
 			(hide yes)

Commit message: layout
Parts:
- C9: footprint Capacitor_SMD:C_0805_2012Metric -> Capacitor_SMD:C_0402_1005Metric
- J1: footprint Connector_USB:USB_Micro-B_Technik_TWP-4002D-H3 -> Connector_USB:USB_Micro-B_Molex_47346-0001
- J2, J3, J4: footprint Connector_PinHeader_1.00mm:PinHeader_1x04_P1.00mm_Vertical_SMD_Pin1Right -> Connector_PinHeader_1.00mm:PinHeader_1x04_P1.00mm_Vertical
Connections:
- net +3.3V: now also J2.1 (Pin_1), J3.1 (Pin_1), J4.1 (Pin_1), R2.1
- net +3.3VA: no longer J2.1 (Pin_1), J3.1 (Pin_1), J4.1 (Pin_1), R2.1
